Commit message: Update ladder-climber urdf to reflect true prismatic joints

File: ladder-climber/description/robot.urdf (robot description, URDF)
Before this commit: robot onshape, 6 links, 5 joints
Joints:
- joint activespring1: type fixed -> prismatic
- joint activespring2: type fixed -> prismatic
- joint passivespring1: type fixed -> prismatic
- joint passivespring2: type fixed -> prismatic
- joint telescope: limit effort=1 velocity=20 -> lower=0 upper=0.7112 effort=1 velocity=20; type fixed -> prismatic

Commit message: working partial ladder climber simulation

File: ladder-climber/description/robot.urdf (robot description, URDF)
Before this commit: robot onshape, 6 links, 5 joints
Links:
- link drivetrain_assembly: mass 259.21 -> 303.881
- link telescoping_hooks_assembly: mass 1.09023 -> 1.36123
Joints:
- joint activespring1: origin xyz=0.009525 0.5715 -2.22045e-16 rpy=1.5708 -9.24446e-33 -6.84228e-49 -> xyz=0.009525 0.5715 6.66134e-16 rpy=1.5708 -9.24446e-33 -6.84228e-49; type prismatic -> fixed
- joint activespring2: origin xyz=0.009525 0 -1.11022e-16 rpy=1.5708 -6.07053e-31 -5.55112e-17 -> xyz=0.009525 0 8.88178e-16 rpy=1.5708 -6.07053e-31 -5.55112e-17; type prismatic -> fixed
- joint passivespring1: origin xyz=0.43815 0.2667 0.889 rpy=1.5708 -2.12635e-17 1.11022e-16 -> xyz=0.43815 0.2667 1.0668 rpy=1.5708 -2.12635e-17 1.11022e-16; type prismatic -> fixed
- joint passivespring2: origin xyz=0.43815 -0.2667 0.889 rpy=-1.5708 -2.12635e-17 -3.14159 -> xyz=0.43815 -0.2667 1.0668 rpy=-1.5708 -2.12635e-17 -3.14159; type prismatic -> fixed
- joint telescope: limit lower=0 upper=0.7112 effort=1 velocity=20 -> lower=0 upper=.889 effort=1 velocity=20; origin xyz=0.43815 -0.28575 0.8382 rpy=-5.12772e-17 2.12635e-17 -4.38764e-42 -> xyz=0.43815 -0.28575 1.016 rpy=-5.12772e-17 2.12635e-17 -4.38764e-42

Commit message: before changing mass

File: ladder-climber/description/robot.urdf (robot description, URDF)
Before this commit: robot onshape, 6 links, 5 joints
Links:
- link passive_hook: geometry collision box size=0.0127 0.0127 0.0635; collision box size=0.0127 0.0127 0.0635
- link passive_hook_2: geometry collision box size=0.0127 0.0127 0.0635; collision box size=0.0127 0.0127 0.0635
- link passive_hook_3: geometry collision box size=0.0127 0.0127 0.0635; collision box size=0.0127 0.0127 0.0635
- link passive_hook_4: geometry collision box size=0.0127 0.0127 0.0635; collision box size=0.0127 0.0127 0.0635
Joints:
- removed joint activespring1
- removed joint activespring2
- removed joint passivespring1
- removed joint passivespring2
- added joint activehook1: type fixed, parent telescoping_hooks_assembly, child passive_hook, origin xyz=0 0.561975 2.22045e-16 rpy=-1.5708 -3.08149e-33 3.14159, axis 0 0 1, limit effort=1 velocity=20
- added joint activehook2: type fixed, parent telescoping_hooks_assembly, child passive_hook_2, origin xyz=-5.55112e-17 -0.009525 4.44089e-16 rpy=-1.5708 -8.51976e-28 -3.14159, axis 0 0 1, limit effort=1 velocity=20
- added joint passivehook1: type revolute, parent drivetrain_assembly, child passive_hook_3, origin xyz=0.43815 0.2667 1.016 rpy=-1.5708 1.4527e-16 -3.33067e-16, axis 0 0 1, limit effort=1 velocity=20
- added joint passivehook2: type revolute, parent drivetrain_assembly, child passive_hook_4, origin xyz=0.43815 -0.3048 1.016 rpy=-1.5708 2.12635e-17 -9.10616e-17, axis 0 0 1, limit effort=1 velocity=20
- joint telescope: limit lower=0 upper=.889 effort=1 velocity=20 -> effort=1 velocity=20; origin xyz=0.43815 -0.28575 1.016 rpy=-5.12772e-17 2.12635e-17 -4.38764e-42 -> xyz=0.43815 -0.28575 1.016 rpy=-5.12772e-17 2.12635e-17 1.03467e-30
